Commit message: removed mesh files from urdf. used simple box shape instead. removed visuals from gazebo model. used the waffle urdf file in urdf directory. documetation and pictures will go into docs/use cases.

File: nav2_system_tests/urdf/turtlebot3_waffle.urdf (robot description, URDF)
Before this commit: robot turtlebot3_waffle, 13 links, 12 joints
Links:
- removed link camera_depth_frame
- removed link camera_link
- added link realsense_depth_frame
- added link realsense_link; collision box size=0.012 0.132 0.020; visual box size=0.1 0.1 0.1
- link base_link: geometry collision box size=0.266 0.266 0.094; visual box size=0.1 0.1 0.1
- link base_scan: geometry collision cylinder length=0.0315 radius=0.055; visual box size=0.1 0.1 0.1
- link wheel_left_link: geometry collision cylinder length=0.018 radius=0.033; visual box size=0.1 0.1 0.1
- link wheel_right_link: geometry collision cylinder length=0.018 radius=0.033; visual box size=0.1 0.1 0.1
Joints:
- removed joint camera_depth_joint
- added joint realsense_depth_joint: type fixed, parent realsense_link, child realsense_depth_frame, origin xyz=0.005 0.028 0.013 rpy=-1.57 0 -1.57
- joint camera_depth_optical_joint: parent camera_depth_frame -> realsense_depth_frame
- joint camera_joint: child camera_link -> realsense_link
- joint camera_rgb_joint: origin xyz=0.005 0.018 0.013 rpy=0 0 0 -> xyz=0.005 0.018 0.013 rpy=-1.57 0 -1.57; parent camera_link -> realsense_link

Commit message: changed robot's shape. used box for the body and cylinder for the wheels, removed realsense references from urdf

File: nav2_system_tests/urdf/turtlebot3_waffle.urdf (robot description, URDF)
Before this commit: robot turtlebot3_waffle, 13 links, 12 joints
Links:
- removed link realsense_depth_frame
- removed link realsense_link
- added link camera_depth_frame
- added link camera_link; collision box size=0.012 0.132 0.020
- link base_link: geometry collision box size=0.266 0.266 0.094; visual box size=0.266 0.266 0.094
- link base_scan: geometry collision cylinder length=0.0315 radius=0.055
- link wheel_left_link: geometry collision cylinder length=0.018 radius=0.033; visual cylinder length=0.018 radius=0.033
- link wheel_right_link: geometry collision cylinder length=0.018 radius=0.033; visual cylinder length=0.018 radius=0.033
Joints:
- removed joint realsense_depth_joint
- added joint camera_depth_joint: type fixed, parent camera_link, child camera_depth_frame, origin xyz=0.005 0.028 0.013 rpy=-1.57 0 -1.57
- joint camera_depth_optical_joint: parent realsense_depth_frame -> camera_depth_frame
- joint camera_joint: child realsense_link -> camera_link
- joint camera_rgb_joint: parent realsense_link -> camera_link
