Commit message: Added more launch files
Signed-off-by: Alejandro Hernández Cordero <ahcorde@gmail.com>

File: nav2_simple_commander/launch/gz_tb3_waffle.urdf (robot description, URDF)
Before this commit: robot turtlebot3_waffle, 13 links, 12 joints
Links:
- link base_link: mass 1.3729096e+00 -> 1.0
- link base_scan: mass 0.114 -> 0.125
- link caster_back_left_link: mass 0.005 -> 0.00001; geometry collision sphere radius=0.005000; visual sphere radius=0.005000
- link caster_back_right_link: mass 0.005 -> 0.001; geometry collision sphere radius=0.005000; visual sphere radius=0.005000
- link wheel_left_link: mass 2.8498940e-02 -> 0.1
- link wheel_right_link: mass 2.8498940e-02 -> 0.1
